File: Hardware/watch-winder/watch-winder.kicad_sch (KiCad schematic)
At the start: 53 parts, among them J1 SWD, J2 UART, J3 MOT, J4 SYNC0, J5 SYNC1, J6 PWR, SW1 SW_Push, SW2 SW_Push, SW3 SW_Push, U1 STM32F030K6Tx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

Commit message: add third mounting hole
Parts:
- removed J2: UART, Connector_PinHeader_2.54mm:PinHeader_1x04_P2.54mm_Horizontal, symbol Connector:Conn_01x04_Pin
- added J2: UART, Connector_PinHeader_2.54mm:PinHeader_1x03_P2.54mm_Vertical, symbol Connector:Conn_01x03_Pin
Connections:
- net +5V: now also J4.3 (Pin_3), J5.3 (Pin_3), J6.2 (Pin_2); no longer J4.1 (Pin_1), J5.1 (Pin_1), J6.1 (Pin_1)
- net GND: now also J4.1 (Pin_1), J5.1 (Pin_1), J6.1 (Pin_1), J2.1 (Pin_1); no longer J4.3 (Pin_3), J5.3 (Pin_3), J6.2 (Pin_2)
- net at R6.2: now also J2.3 (Pin_3)
- net at R5.2: now also J2.2 (Pin_2)
Other:
- moved on the sheet: J6, R10, R11, R12, R13, R5, R6
